Commit message: fixed axis issue, fucking end effector issue is still there. fuck you solidworks

File: gp7_robot/urdf/gp7_robot.urdf (robot description, URDF)
Before this commit: robot gp7_robot, 9 links, 8 joints
Links:
- link finger2_link: mass 0.02604 -> 0.026039744934362
- link link2: mass 6.2406 -> 6.2405
- link link3: mass 2.8491 -> 2.8492
Joints:
- joint finger1_joint: axis 0.040132 0 0.99919 -> 0.0401317925325461 0 -0.999194395114446; origin xyz=-0.015003 0.024747 0.10859 rpy=1.5602 -0.25861 2.4732 -> xyz=-0.0263403229325416 0.0119878501740266 0.10858504415831 rpy=1.51758990402072 -0.923956186840669 3.09700319298282
- joint finger2_joint: axis 0.040132 0 0.99919 -> 0.040132 0 -0.99919; origin xyz=0.013688 -0.025498 0.10859 rpy=1.5757 0.12207 -0.72183 -> xyz=0.025677 -0.01335 0.10859 rpy=1.5176 -0.92396 -0.096949
- joint joint1: axis 0 0 1 -> 0 0 -1; origin xyz=-0.00059534 0 0.1829 rpy=0 0 0 -> xyz=-0.000595342695521883 0 0.1829 rpy=0 0 0
- joint joint2: axis 0 0 1 -> 0 0 -1; origin xyz=-0.022744 -0.079163 0.1355 rpy=1.3435 -1.5708 0 -> xyz=0.0481152180218847 0.0668500247537757 0.135500000000094 rpy=1.57079632679473 0 3.0248336337098
- joint joint3: axis 0 0 1 -> 0 0 -1; origin xyz=0.34163 0.28515 0 rpy=0 0 3.1416 -> xyz=0.166975951159858 0.412485189717141 0 rpy=0 0 -1.57079632679492
- joint joint4: axis 0.31036 0 0.95062 -> 0 0 -1; origin xyz=-0.062543 -0.062685 -0.072 rpy=1.5708 0 0 -> xyz=-0.00319297470642954 -0.0884918352576554 -0.0720000000000005 rpy=-1.57079632679483 -0.272786020633957 -2.70896107573833
- joint joint5: axis 0 0 1 -> 0 0 -1; origin xyz=-0.11212 -0.0135 0.34315 rpy=1.5735 -0.80813 -0.0076134 -> xyz=-0.00132428368504911 0.0134348901237163 0.361000000001776 rpy=1.57079632679489 0.0421986683723227 -3.04333955815242
- joint joint6: origin xyz=0 0.0675 -0.0135 rpy=1.5708 1.5626 -3.1416 -> xyz=0 0.0674999999997865 -0.0134999999999023 rpy=1.57079632697687 1.39265583816902 -3.14159265335474
