Commit message: all working after urdf update

File: gp7_robot/gp7_robot_w.urdf (robot description, URDF)
Before this commit: robot gp7_robot, 10 links, 9 joints
Links:
- link finger2_link: mass 0.0047666 -> 0.00476659381411143
Joints:
- joint finger1_joint: axis 0.0012983 0.14877 0.98887 -> 0 1 0; limit lower=-1 upper=0.5 effort=10 velocity=2.0 -> lower=-0.7 upper=0.7 effort=10 velocity=2.0; origin xyz=-0.0074919 0.012828 -0.1675 rpy=-1.5708 1.5621 1.5708 -> xyz=-0.012828 0.0074919 0.1 rpy=1.5708 -1.5621 3.14
- joint finger2_joint: axis -0.0012983 -0.14877 -0.98887 -> 0 -1 0; limit lower=-1 upper=0.5 effort=10 velocity=2.0 -> lower=-0.7 upper=0.7 effort=10 velocity=2.0; origin xyz=-0.0033856 -0.014465 -0.1675 rpy=-1.5708 1.5621 1.5708 -> xyz=0.014465 0.0033856 0.1 rpy=1.5708 -1.5621 3.14
- joint joint3: axis 0 0 -1 -> -0 -0 -1
- joint joint4: origin xyz=-0.04 0 0.00062392 rpy=1.5708 0 0 -> xyz=-0.04 -0.079 0 rpy=1.5708 1.5708 0
- joint joint5: origin xyz=0 -0.00062392 0.43999 rpy=-1.5708 0 0 -> xyz=0 0 0.361 rpy=1.5708 0 -1.5708
- joint joint6: origin xyz=0 0 0 rpy=-1.5708 0 0 -> xyz=0 0.0675 0 rpy=-1.5708 1.5708 0
