Commit message: gazebo spawning okay

File: src/gp7_robot/urdf/gp7_robot.urdf (robot description, URDF)
Before this commit: robot gp7_robot, 9 links, 8 joints
Links:
- removed link finger1_link
- removed link finger2_link
- added link world
Joints:
- removed joint finger1_joint
- removed joint finger2_joint
- added joint world_to_base: type fixed, parent world, child base_link, origin xyz=0 0 0 rpy=0 0 0

Commit message: issues with urdf still exist. fix

File: src/gp7_robot/urdf/gp7_robot.urdf (robot description, URDF)
Before this commit: robot gp7_robot, 8 links, 7 joints
Links:
- added link finger1_link, mass 0.0047666; collision mesh filename=package://gp7_robot/meshes/finger1_link.STL; visual mesh filename=package://gp7_robot/meshes/finger1_link.STL
- added link finger2_link, mass 0.00476659381411143; collision mesh filename=package://gp7_robot/meshes/finger2_link.STL; visual mesh filename=package://gp7_robot/meshes/finger2_link.STL
- link EE: mass 0.12078 -> 0.13667
Joints:
- added joint finger1_joint: type revolute, parent EE, child finger1_link, origin xyz=-0.012828 0.0074919 0.1 rpy=1.5708 -1.5621 -3.1416, axis 0.0012983 0.14877 0.98887, limit lower=0 upper=0 effort=0 velocity=0
- added joint finger2_joint: type revolute, parent EE, child finger2_link, origin xyz=0.014465 0.0033856 0.1 rpy=1.5708 -1.5621 -3.1416, axis 0.0012983 0.14877 0.98887, limit lower=0 upper=0 effort=0 velocity=0
- joint joint1: origin xyz=-0.000595342695521883 0 0.1829 rpy=0 0 0 -> xyz=-0.00059534 0 0.1829 rpy=0 0 0
- joint joint2: origin xyz=0.0481152180218847 0.0668500247537757 0.135500000000094 rpy=1.57079632679473 0 3.0248336337098 -> xyz=0.039998 0.00034906 0.1355 rpy=1.5708 0 -3.1329
- joint joint3: origin xyz=0.166975951159858 0.412485189717141 0 rpy=0 0 -1.57079632679492 -> xyz=0 0.445 0 rpy=0 0 -1.5708
- joint joint4: origin xyz=-0.00319297470642954 -0.0884918352576554 -0.0720000000000005 rpy=-1.57079632679483 -0.272786020633957 -2.70896107573833 -> xyz=-0.04 -0.079 0 rpy=1.5708 1.5708 0
- joint joint5: origin xyz=-0.00132428368504911 0.0134348901237163 0.361000000001776 rpy=1.57079632679489 0.0421986683723227 -3.04333955815242 -> xyz=0 0 0.361 rpy=1.5708 0 -1.5708
- joint joint6: origin xyz=0 0.0674999999997865 -0.0134999999999023 rpy=1.57079632697687 1.39265583816902 -3.14159265335474 -> xyz=0 0.0675 0 rpy=1.5708 -1.5708 0

Commit message: controllers working. but found out one frame assignment isn't correct. need to go back to solidwork and come back

File: src/gp7_robot/urdf/gp7_robot.urdf (robot description, URDF)
Before this commit: robot gp7_robot, 10 links, 9 joints
Links:
- link finger1_link: geometry collision box size=0.015 0.01 0.04; visual mesh filename=package://gp7_robot/meshes/finger1_link.STL
- link finger2_link: geometry collision box size=0.015 0.01 0.04; visual mesh filename=package://gp7_robot/meshes/finger2_link.STL
Joints:
- joint finger1_joint: axis 0.0012983 0.14877 0.98887 -> 0 1 0; limit lower=0 upper=0 effort=0 velocity=0 -> lower=-0.7 upper=0.7 effort=10 velocity=2.0; origin xyz=-0.012828 0.0074919 0.1 rpy=1.5708 -1.5621 -3.1416 -> xyz=-0.012828 0.0074919 0.1 rpy=1.5708 -1.5621 3.14
- joint finger2_joint: axis 0.0012983 0.14877 0.98887 -> 0 -1 0; limit lower=0 upper=0 effort=0 velocity=0 -> lower=-0.7 upper=0.7 effort=10 velocity=2.0; origin xyz=0.014465 0.0033856 0.1 rpy=1.5708 -1.5621 -3.1416 -> xyz=0.014465 0.0033856 0.1 rpy=1.5708 -1.5621 3.14
- joint joint1: limit lower=-2.96706 upper=2.96706 effort=0 velocity=6.54499 -> lower=-2.96706 upper=2.96706 effort=200 velocity=6.54499
- joint joint2: limit lower=-1.13446 upper=2.53073 effort=0 velocity=5.49779 -> lower=-1.13446 upper=2.53073 effort=200 velocity=5.49779
- joint joint3: axis 0 0 1 -> -0 -0 -1; limit lower=-1.22173 upper=3.31613 effort=0 velocity=7.15585 -> lower=-1.22173 upper=3.31613 effort=200 velocity=7.15585
- joint joint4: limit lower=-3.31613 upper=3.31613 effort=0 velocity=9.59931 -> lower=-3.31613 upper=3.31613 effort=17 velocity=9.59931
- joint joint5: limit lower=-2.35619 upper=2.35619 effort=0 velocity=9.59931 -> lower=-2.35619 upper=2.35619 effort=17 velocity=9.59931
- joint joint6: limit (none) -> lower=-6.28318 upper=6.28318 effort=10 velocity=17.4533; origin xyz=0 0.0675 0 rpy=1.5708 -1.5708 0 -> xyz=0 0.0675 0 rpy=-1.5708 1.5708 0

Commit message: issues exist

File: src/gp7_robot/urdf/gp7_robot.urdf (robot description, URDF)
Before this commit: robot gp7_robot, 10 links, 9 joints
Joints:
- joint joint3: axis 0 0 -1 -> 0 0 1
- joint joint4: limit lower=-3.31613 upper=3.31613 effort=17 velocity=9.59931 -> lower=-3.31613 upper=3.31613 effort=50 velocity=9.59931
- joint joint5: limit lower=-2.35619 upper=2.35619 effort=17 velocity=9.59931 -> lower=-2.35619 upper=2.35619 effort=50 velocity=9.59931
- joint joint6: limit lower=-6.28318 upper=6.28318 effort=10 velocity=17.4533 -> lower=-6.28318 upper=6.28318 effort=20 velocity=17.4533

Commit message: fixed DH again, but gpt says its still wrong according to urdf

File: src/gp7_robot/urdf/gp7_robot.urdf (robot description, URDF)
Before this commit: robot gp7_robot, 10 links, 9 joints
Joints:
- joint joint4: limit lower=-3.31613 upper=3.31613 effort=50 velocity=9.59931 -> lower=-3.31613 upper=3.31613 effort=17 velocity=9.59931
- joint joint5: limit lower=-2.35619 upper=2.35619 effort=50 velocity=9.59931 -> lower=-2.35619 upper=2.35619 effort=17 velocity=9.59931
- joint joint6: limit lower=-6.28318 upper=6.28318 effort=20 velocity=17.4533 -> lower=-6.28318 upper=6.28318 effort=10 velocity=17.4533
